File: monKWH-RS485/untitled.sch (EAGLE design)
At the start: 49 parts, among them J1 U.FL-R-SMT(01), J2 DCJ0202, J3 10103594, Q1 MMBT3904, Q2 MMBT3904, Q3 12MHz, U1 RT9193-33GB, U2 RT9193-33GB, X1 MSTBA2, X2 MSTBA2

Commit message: PCBv1.0
Connections:
- net 3V3: now also R4.2, R5.2
- net VCC: no longer R4.2, R5.2
Changed lines of the file:
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@@
 <part name="GND4" library="supply1" library_urn="urn:adsk.eagle:library:371" deviceset="GND" device=""/>
 <part name="D4" library="1N5819HW-7" deviceset="1N5819HW-7" device=""/>
-<part name="P+1" library="supply1" library_urn="urn:adsk.eagle:library:371" deviceset="VCC" device=""/>
 <part name="P+3" library="supply1" library_urn="urn:adsk.eagle:library:371" deviceset="VCC" device=""/>
 <part name="MD1" library="Espressif Systems - ESP32-WROOM-32U (16MB)" deviceset="ESPRESSIF_SYSTEMS_ESP32-WROOM-32U_16MB" device="ESPRESSIF_SYSTEMS_ESP32-WROOM-32U_16MB_0_0"/>
@@
 <attribute name="VALUE" x="93.98" y="158.75" size="1.778" layer="96"/>
 </instance>
-<instance part="P+1" gate="VCC" x="68.58" y="55.88" smashed="yes">
-<attribute name="VALUE" x="66.04" y="53.34" size="1.778" layer="96" rot="R90"/>
-</instance>
 <instance part="P+3" gate="VCC" x="-76.2" y="116.84" smashed="yes" rot="R180">
 <attribute name="VALUE" x="-73.66" y="119.38" size="1.778" layer="96" rot="R270"/>
@@
 <junction x="88.9" y="121.92"/>
 </segment>
+<segment>
+<pinref part="R4" gate="G$1" pin="2"/>
+<pinref part="R5" gate="G$1" pin="2"/>
+<wire x1="66.04" y1="48.26" x2="68.58" y2="48.26" width="0.1524" layer="91"/>
+<wire x1="68.58" y1="48.26" x2="71.12" y2="48.26" width="0.1524" layer="91"/>
+<junction x="68.58" y="48.26"/>
+<wire x1="68.58" y1="53.34" x2="68.58" y2="48.26" width="0.1524" layer="91"/>
+<label x="68.58" y="53.34" size="1.778" layer="95" rot="R90" xref="yes"/>
+</segment>
 </net>
 <net name="N$12" class="0">
@@
 <net name="VCC" class="0">
 <segment>
-<pinref part="R4" gate="G$1" pin="2"/>
-<pinref part="R5" gate="G$1" pin="2"/>
-<wire x1="66.04" y1="48.26" x2="68.58" y2="48.26" width="0.1524" layer="91"/>
-<wire x1="68.58" y1="48.26" x2="71.12" y2="48.26" width="0.1524" layer="91"/>
-<junction x="68.58" y="48.26"/>
-<pinref part="P+1" gate="VCC" pin="VCC"/>
-<wire x1="68.58" y1="53.34" x2="68.58" y2="48.26" width="0.1524" layer="91"/>
-</segment>
-<segment>
 <pinref part="C1" gate="G$1" pin="1"/>
